File: 675-fan-ctl/675-fan-ctl.sch (KiCad schematic (older format))
At the start: 15 parts, among them J1 +, J2 -, J3 M+, J4 M-, Q1 3055T, SW1 High Spin, U1 LM7805_TO220, U2 PIC12F675-IP

Commit message: small changes.
Parts:
- added J5, J6: Conn_01x01_Male, Connectors:Pin_d1.4mm_L8.5mm_W2.8mm_FlatFork, symbol Connector:Conn_01x01_Male
Connections:
- wire segments 39 -> 42
- no-connect marks 3 -> 1
Changed lines of the file:
@@
 Wire Wire Line
 	5350 2950 5350 2850
-NoConn ~ 5100 3050
 $Comp
 L Device:Thermistor_NTC TH1
@@
 	5850 2850 5850 2700
 NoConn ~ 3900 2950
-NoConn ~ 3900 3150
 Wire Wire Line
 	6800 3650 6400 3650
@@
 Wire Wire Line
 	3900 3050 3600 3050
+$Comp
+L Connector:Conn_01x01_Male J6
+U 1 1 5B7496BC
+P 5400 3900
+F 0 "J6" H 5373 3830 50  0000 R CNN
+F 1 "Conn_01x01_Male" H 5373 3921 50  0000 R CNN
+F 2 "Connectors:Pin_d1.4mm_L8.5mm_W2.8mm_FlatFork" H 5400 3900 50  0001 C CNN
+F 3 "~" H 5400 3900 50  0001 C CNN
+	1    5400 3900
+	-1   0    0    1
+$EndComp
+$Comp
+L Connector:Conn_01x01_Male J5
+U 1 1 5B7498D6
+P 3700 3900
+F 0 "J5" H 3806 4078 50  0000 C CNN
+F 1 "Conn_01x01_Male" H 3806 3987 50  0000 C CNN
+F 2 "Connectors:Pin_d1.4mm_L8.5mm_W2.8mm_FlatFork" H 3700 3900 50  0001 C CNN
+F 3 "~" H 3700 3900 50  0001 C CNN
+	1    3700 3900
+	1    0    0    -1
+$EndComp
+Wire Wire Line
+	3900 3150 3900 3900
+Wire Wire Line
+	5100 3050 5200 3050
+Wire Wire Line
+	5200 3050 5200 3900
 $EndSCHEMATC

Commit message: add capacitor.
Parts:
- added C4: 47u, Capacitors_THT:CP_Radial_D6.3mm_P2.50mm, symbol Device:CP
Connections:
- wire segments 42 -> 45
Changed lines of the file:
@@
 Wire Wire Line
 	5200 3050 5200 3900
+$Comp
+L Device:CP C4
+U 1 1 5B74D34C
+P 2000 2700
+F 0 "C4" H 2118 2746 50  0000 L CNN
+F 1 "47u" H 2118 2655 50  0000 L CNN
+F 2 "Capacitors_THT:CP_Radial_D6.3mm_P2.50mm" H 2038 2550 50  0001 C CNN
+F 3 "~" H 2000 2700 50  0001 C CNN
+	1    2000 2700
+	1    0    0    -1
+$EndComp
+Wire Wire Line
+	2000 2850 2000 3000
+Wire Wire Line
+	2000 3000 2700 3000
+Wire Wire Line
+	2000 2550 2000 2450
+Connection ~ 2000 2450
 $EndSCHEMATC
